File: FlashyButton/FlashyButton.kicad_pcb (KiCad board)
At the start: 2 copper layers, 24 x 22 mm, 9 parts, among them J1 Conn_01x04_Pin, SW1 SW_Push, SW2 SW_Push

Commit message: Pushed flashybutton to mfg
Parts:
- removed the REF** at (175.3, 105.1)
- removed the REF** at (157.5, 105.2)
- removed the REF** at (175.4, 89.2)
- added REF**: MountingHole_2.7mm_M2.5_DIN965_Pad, MountingHole:MountingHole_2.7mm_M2.5_DIN965_Pad, F.Cu at (175.3, 105.1)
- added REF**: MountingHole_2.7mm_M2.5_DIN965_Pad, MountingHole:MountingHole_2.7mm_M2.5_DIN965_Pad, F.Cu at (157.5, 105.2)
- added REF**: MountingHole_2.7mm_M2.5_DIN965_Pad, MountingHole:MountingHole_2.7mm_M2.5_DIN965_Pad, F.Cu at (175.4, 89.2)
Routing:
- net /Power: track 13.9 -> 0.00 mm
- added copper zone on F.Cu, net /Power
Changed lines of the file:
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@@
 		)
 	)
-	(footprint "MountingHole:MountingHole_2.7mm_M2.5"
+	(footprint "MountingHole:MountingHole_2.7mm_M2.5_DIN965_Pad"
 		(layer "F.Cu")
 		(at 175.3108 105.1306)
-		(descr "Mounting Hole 2.7mm, M2.5, no annular, generated by kicad-footprint-generator mountinghole.py")
-		(tags "mountinghole M2.5")
+		(descr "Mounting Hole 2.7mm, M2.5, generated by kicad-footprint-generator mountinghole.py")
+		(tags "mountinghole M2.5 DIN965")
 		(property "Reference" "REF**"
-			(at 0 -3.65 0)
+			(at 0 -3.3 0)
 			(layer "F.SilkS")
 			(hide yes)
@@
 			)
 		)
-		(property "Value" "MountingHole_2.7mm_M2.5"
-			(at 0 3.65 0)
+		(property "Value" "MountingHole_2.7mm_M2.5_DIN965_Pad"
+			(at 0 3.3 0)
 			(layer "F.Fab")
 			(effects
@@
 		(fp_circle
 			(center 0 0)
-			(end 2.7 0)
+			(end 2.35 0)
 			(stroke
 				(width 0.15)
@@
 		(fp_circle
 			(center 0 0)
-			(end 2.95 0)
+			(end 2.6 0)
 			(stroke
 				(width 0.05)
@@
 			)
 		)
-		(pad "" np_thru_hole circle
+		(pad "1" thru_hole circle
 			(at 0 0)
-			(size 2.7 2.7)
+			(size 4.7 4.7)
 			(drill 2.7)
 			(layers "*.Cu" "*.Mask")
+			(remove_unused_layers no)
+			(zone_connect 2)
+		)
+		(embedded_fonts no)
+	)
+	(footprint "MountingHole:MountingHole_2.7mm_M2.5_DIN965_Pad"
+		(layer "F.Cu")
+		(at 157.4546 105.1814)
+		(descr "Mounting Hole 2.7mm, M2.5, generated by kicad-footprint-generator mountinghole.py")
+		(tags "mountinghole M2.5 DIN965")
+		(property "Reference" "REF**"
+			(at 0 -3.3 0)
+			(layer "F.SilkS")
+			(hide yes)
+			(effects
+				(font
+					(size 1 1)
+					(thickness 0.15)
+				)
+			)
+		)
+		(property "Value" "MountingHole_2.7mm_M2.5_DIN965_Pad"
+			(at 0 3.3 0)
+			(layer "F.Fab")
+			(effects
+				(font
+					(size 1 1)
+					(thickness 0.15)
+				)
+			)
+		)
+		(property "Datasheet" ""
+			(at 0 0 0)
+			(layer "F.Fab")
+			(hide yes)
+			(effects
+				(font
+					(size 1.27 1.27)
+				)
+			)
+		)
+		(property "Description" ""
+			(at 0 0 0)
+			(layer "F.Fab")
+			(hide yes)
+			(effects
+				(font
+					(size 1.27 1.27)
+				)
+			)
+		)
+		(property "KiLib_Generator" "mounting_hardware/mounting_hole"
+			(at 0 0 0)
+			(layer "F.SilkS")
+			(hide yes)
+			(effects
+				(font
+					(size 1 1)
+					(thickness 0.15)
+				)
+			)
+		)
+		(attr exclude_from_pos_files exclude_from_bom)
+		(duplicate_pad_numbers_are_jumpers no)
+		(fp_circle
+			(center 0 0)
+			(end 2.35 0)
+			(stroke
+				(width 0.15)
+				(type solid)
+			)
+			(fill no)
+			(layer "Cmts.User")
+		)
+		(fp_circle
+			(center 0 0)
+			(end 2.6 0)
+			(stroke
+				(width 0.05)
+				(type solid)
+			)
+			(fill no)
+			(layer "F.CrtYd")
+		)
+		(fp_text user "${REFERENCE}"
+			(at 0 0 0)
+			(layer "F.Fab")
+			(effects
+				(font
+					(size 1 1)
+					(thickness 0.15)
+				)
+			)
+		)
+		(pad "1" thru_hole circle
+			(at 0 0)
+			(size 4.7 4.7)
+			(drill 2.7)
+			(layers "*.Cu" "*.Mask")
+			(remove_unused_layers no)
+			(zone_connect 2)
 		)
 		(embedded_fonts no)
@@
 		)
 	)
-	(footprint "MountingHole:MountingHole_2.7mm_M2.5"
+	(footprint "MountingHole:MountingHole_2.7mm_M2.5_DIN965_Pad"
 		(layer "F.Cu")
-		(at 157.4546 105.1814)
-		(descr "Mounting Hole 2.7mm, M2.5, no annular, generated by kicad-footprint-generator mountinghole.py")
-		(tags "mountinghole M2.5")
+		(at 175.4 89.2)
+		(descr "Mounting Hole 2.7mm, M2.5, generated by kicad-footprint-generator mountinghole.py")
+		(tags "mountinghole M2.5 DIN965")
 		(property "Reference" "REF**"
-			(at 0 -3.65 0)
+			(at 0 -3.3 0)
 			(layer "F.SilkS")
 			(hide yes)
@@
 			)
 		)
-		(property "Value" "MountingHole_2.7mm_M2.5"
-			(at 0 3.65 0)
+		(property "Value" "MountingHole_2.7mm_M2.5_DIN965_Pad"
+			(at 0 3.3 0)
 			(layer "F.Fab")
 			(effects
@@
 		(fp_circle
 			(center 0 0)
-			(end 2.7 0)
+			(end 2.35 0)
 			(stroke
 				(width 0.15)
@@
 		(fp_circle
 			(center 0 0)
-			(end 2.95 0)
+			(end 2.6 0)
 			(stroke
 				(width 0.05)
@@
 			)
 		)
-		(pad "" np_thru_hole circle
-			(at 0 0)
-			(size 2.7 2.7)
-			(drill 2.7)
-			(layers "*.Cu" "*.Mask")
-		)
-		(embedded_fonts no)
-	)
-	(footprint "MountingHole:MountingHole_2.7mm_M2.5"
-		(layer "F.Cu")
-		(at 175.387 89.154)
-		(descr "Mounting Hole 2.7mm, M2.5, no annular, generated by kicad-footprint-generator mountinghole.py")
-		(tags "mountinghole M2.5")
-		(property "Reference" "REF**"
-			(at 0 -3.65 0)
-			(layer "F.SilkS")
-			(hide yes)
-			(effects
-				(font
-					(size 1 1)
-					(thickness 0.15)
-				)
-			)
-		)
-		(property "Value" "MountingHole_2.7mm_M2.5"
-			(at 0 3.65 0)
-			(layer "F.Fab")
-			(effects
-				(font
-					(size 1 1)
-					(thickness 0.15)
-				)
-			)
-		)
-		(property "Datasheet" ""
-			(at 0 0 0)
-			(layer "F.Fab")
-			(hide yes)
-			(effects
-				(font
-					(size 1.27 1.27)
-				)
-			)
-		)
-		(property "Description" ""
-			(at 0 0 0)
-			(layer "F.Fab")
-			(hide yes)
-			(effects
-				(font
-					(size 1.27 1.27)
-				)
-			)
-		)
-		(property "KiLib_Generator" "mounting_hardware/mounting_hole"
-			(at 0 0 0)
-			(layer "F.SilkS")
-			(hide yes)
-			(effects
-				(font
-					(size 1 1)
-					(thickness 0.15)
-				)
-			)
-		)
-		(attr exclude_from_pos_files exclude_from_bom)
-		(duplicate_pad_numbers_are_jumpers no)
-		(fp_circle
-			(center 0 0)
-			(end 2.7 0)
-			(stroke
-				(width 0.15)
-				(type solid)
-			)
-			(fill no)
-			(layer "Cmts.User")
-		)
-		(fp_circle
-			(center 0 0)
-			(end 2.95 0)
-			(stroke
-				(width 0.05)
-				(type solid)
-			)
-			(fill no)
-			(layer "F.CrtYd")
-		)
-		(fp_text user "${REFERENCE}"
-			(at 0 0 0)
-			(layer "F.Fab")
-			(effects
-				(font
-					(size 1 1)
-					(thickness 0.15)
-				)
-			)
-		)
-		(pad "" np_thru_hole circle
+		(pad "1" thru_hole circle
 			(at 0 0)
-			(size 2.7 2.7)
+			(size 4.7 4.7)
 			(drill 2.7)
 			(layers "*.Cu" "*.Mask")
+			(remove_unused_layers no)
+			(zone_connect 2)
 		)
 		(embedded_fonts no)
@@
 	)
 	(gr_text "5v"
-		(at 162.941 91.0082 90)
+		(at 162.8 92.6 0)
 		(layer "B.SilkS")
 		(effects
 			(font
-				(size 1.2 1.2)
+				(size 1 1)
 				(bold yes)
 			)
@@
 	)
 	(gr_text "LED"
-		(at 165.227 91.0082 90)
+		(at 165.8 92.6 0)
 		(layer "B.SilkS")
 		(effects
 			(font
-				(size 1.2 1.2)
+				(size 1 1)
 				(bold yes)
 			)
@@
 	)
 	(gr_text "GND"
-		(at 167.894 90.8812 90)
+		(at 169 92.6 0)
 		(layer "B.SilkS")
 		(effects
 			(font
-				(size 1.2 1.2)
+				(size 1 1)
 				(bold yes)
 			)
@@
 	)
 	(gr_text "BTN"
-		(at 170.561 89.3572 180)
+		(at 172 92.6 0)
 		(layer "B.SilkS")
 		(effects
 			(font
-				(size 1.2 1.2)
+				(size 1 1)
 				(bold yes)
 			)
@@
 	)
 	(segment
-		(start 163.576 99.7712)
-		(end 162.814 99.7712)
-		(width 0.6)
-		(layer "F.Cu")
-		(net "/Power")
-	)
-	(segment
-		(start 160.02 91.3892)
-		(end 159.033 91.3892)
-		(width 0.6)
-		(layer "F.Cu")
-		(net "/Power")
-	)
-	(segment
-		(start 162.814 99.7712)
-		(end 162.433 99.3902)
-		(width 0.6)
-		(layer "F.Cu")
-		(net "/Power")
-	)
-	(segment
-		(start 160.274 91.6432)
-		(end 160.02 91.3892)
-		(width 0.6)
-		(layer "F.Cu")
-		(net "/Power")
-	)
-	(segment
-		(start 162.433 92.6592)
-		(end 162.052 92.2782)
-		(width 0.6)
-		(layer "F.Cu")
-		(net "/Power")
-	)
-	(segment
-		(start 162.052 92.2782)
-		(end 162.052 91.6432)
-		(width 0.6)
-		(layer "F.Cu")
-		(net "/Power")
-	)
-	(segment
-		(start 162.052 91.6432)
-		(end 162.052 90.1192)
-		(width 0.6)
-		(layer "F.Cu")
-		(net "/Power")
-	)
-	(segment
-		(start 162.052 91.6432)
-		(end 160.274 91.6432)
-		(width 0.6)
-		(layer "F.Cu")
-		(net "/Power")
-	)
-	(segment
-		(start 162.433 99.3902)
-		(end 162.433 92.6592)
-		(width 0.6)
-		(layer "F.Cu")
-		(net "/Power")
-	)
-	(segment
 		(start 163.576 93.6752)
 		(end 164.592 92.6592)
@@
 	)
 	(zone
+		(net "/Power")
+		(layer "F.Cu")
+		(hatch edge 0.5)
+		(priority 1)
+		(connect_pads yes
+			(clearance 0.2)
+		)
+		(min_thickness 0.25)
+		(fill yes
+			(thermal_gap 0.5)
+			(thermal_bridge_width 0.5)
+			(smoothing fillet)
+			(radius 1)
+			(island_removal_mode 0)
+		)
+		(polygon
+			(pts
+				(xy 161 90.5192) (xy 158.4 90.5192) (xy 158.4 92.4) (xy 162.052 92.4) (xy 162.052 100.6) (xy 164.2 100.6)
+				(xy 164.2 98.8) (xy 163 98.8) (xy 163 89.2) (xy 161 89.2)
+			)
+		)
+	)
+	(zone
