File: SparkleBoard/sparkleboard5v.kicad_sch (KiCad schematic)
At the start: 33 parts, among them J3 Conn_01x04_Pin, J4 Conn_01x02_Pin, J5 Conn_01x02_Pin, U1 C9900066641, U2 AONR21307, U3 HUSB238, U6 AP63205WU

Commit message: redesigned board around HUSB238*A*. Pin compatible, but non-A revision seems to be EOL. HUSB238A has different footprint (QFN?) Enlarged board to make more logical groupings of components (ie ISET/VSET) USB connector (C9900066641) is also EOL and should be replaced before MFG
Parts:
- removed R3: 10, Resistor_SMD:R_0603_1608Metric, symbol PCM_SparkFun-Resistor:100k_0603
- removed U3: HUSB238, EasyEDA_Lib:TDFN-10_L3.0-W3.0-P0.50-TL-EP, symbol EasyEDA_Lib:HUSB238
- added R11: 900k, Resistor_SMD:R_0805_2012Metric, symbol PCM_SparkFun-Resistor:100k_0603
- added U4: HUSB238A-xxxxx-QN16R, Package_DFN_QFN:WQFN-16-1EP_3x3mm_P0.5mm_EP1.75x1.75mm, symbol Interface_USB:HUSB238A-xxxxx-QN16R
- C12: footprint Capacitor_SMD:C_1210_3225Metric -> Capacitor_SMD:C_0805_2012Metric
- J3: footprint Connector_PinHeader_2.54mm:PinHeader_1x04_P2.54mm_Vertical -> EasyEDA_Lib:CONN-TH_DB125-2.54-4P-GN
- R10, R5, R6, R7, R9: footprint Resistor_SMD:R_0603_1608Metric -> Resistor_SMD:R_0805_2012Metric
Connections:
- net CC1: now also U4.3 (CC1)
- net CC2: now also U4.4 (CC2)
- net GND: now also U1.EH1, R11.1, U4.17 (GND)
- net ISET: now also U4.10 (SCL/SNK_ISET)
- net USBC_D+: now also U4.1 (D+)
- net USBC_D-: now also U4.2 (D-)
- net VBUS: now also C14.2, U4.16 (VBUS)
- net VSET: now also U4.9 (SDA/SNK_VSET)
- net at R10.1: now also U4.15 (GATE)
- new net: R11.2, U4.6 (~{DEBUG})
- no-connect marks 4 -> 8
Other:
- note added: "EN_HVDCP/OUT1 is for BC2.1 (Battery Charging)"
- moved on the sheet: C12, C13, C14, C20, C21, L1, R1, R2, R9, U6
